File: claude-code-pad/pcb/claude-code-pad.kicad_pcb (KiCad board)
At the start: 2 copper layers, 120 x 134 mm, 137 parts, among them SW00 MX_HS, SW01 MX_HS, SW02 MX_HS, SW03 MX_HS, SW04 MX_HS, SW10 MX_HS, SW11 MX_HS, SW12 MX_HS, SW13 MX_HS, SW14 MX_HS, SW20 MX_HS, SW21 MX_HS, SW22 MX_HS, SW23 MX_HS, SW24 MX_HS, SW30 MX_HS, SW31 MX_HS, SW32 MX_HS, SW33 MX_HS, SW34 MX_HS, SW40 MX_HS, SW41 MX_HS, SW42 MX_HS, SW43 MX_HS, SW44 MX_HS, U1 XIAO_nRF52840

Commit message: Close Phase 1 PCB: Freerouting pipeline + mandatory battery docs
Across cycles 2-7, drove the PCB through adversarial review to a
fab-ready state. Major decisions logged in docs/review-log.md:

- Scope: dropped TinyML + SSD1306 OLED; swapped ESP32-S3 → nRF52840
  (ZMK-native, retires Phase 4 and ML-1 persona).
- Power: simplified to XIAO on-module charger + DMG3415U reverse-pol
  FET + 500 mA PTC + firmware LED cap per IEC 62368-1 Annex Q, after
  a discrete PCM+charger+mux+buck iteration produced multiple
  pinout errors.
- Routing: generative-Python routing abandoned; installed Freerouting
  2.1.0 in the kicad distrobox for headless autoroute. 1095 routed
  segments, 148 GND stitching vias, antenna keepout inviolate,
  Power netclass widened to 0.80 mm post-SES.
- Layout: board 120 x 132 mm (up from 115 x 105 to accommodate MCU,
  encoder, stabilized 2U Enter, antenna keepout). 2U east stab
  clearance resolved by board width bump.
- Safety: cell-level PCM delegation documented as MANDATORY in
  docs/build-guide.md with verified Adafruit/SparkFun LCSC cells;
  JST-SH -> JST-PH migration acknowledged throughout.

Workflow change: pcb/_gen/generate.py now produces footprints +
schematic + placement only. Routing lives in the .kicad_pcb after
Freerouting. Regenerating from the generator destroys routing.

Added at repo root:
- README.md: project orientation + Bazzite tooling conventions.
- CLAUDE.md: KiCad flatpak invocation, distrobox setup, KiCad-MCP
  registration, host/container version skew notes.
- .mcp.json: auto-loads lamaalrajih/kicad-mcp from the distrobox.
- .gitignore: KiCad lockfiles, .history/, __pycache__/.

Phase 1 closed after Cycle 7; Cycle 8 (GUI-DRC cleanup for
hole_clearance on CL caps + UUID linkage) is in progress.

Co-Authored-By: Claude Opus 4.7 (1M context) <noreply@anthropic.com>
Parts:
- moved D00 4.00 mm to (123.4, 144.5)
- moved D02 4.00 mm to (161.5, 144.5)
- moved D03 4.00 mm to (180.6, 144.5)
- moved D10 4.00 mm to (123.4, 163.6)
- moved D12 4.00 mm to (161.5, 163.6)
- moved D13 4.00 mm to (180.6, 163.6)
- moved D20 4.00 mm to (123.4, 182.6)
- moved D22 4.00 mm to (161.5, 182.6)
- moved D23 4.00 mm to (180.6, 182.6)
- moved D30 4.00 mm to (123.4, 201.7)
- moved D32 4.00 mm to (161.5, 201.7)
- moved D33 4.00 mm to (180.6, 201.7)
- moved D40 4.00 mm to (123.4, 220.7)
- moved D42 4.00 mm to (161.5, 220.7)
- moved D43 4.00 mm to (180.6, 220.7)
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Connections:
- J_XIAO_BP pad 4: ROW3 -> RGB_DIN_MCU
- J_XIAO_BP pad 5: ROW4 -> ROW3
- J_XIAO_BP pad 6: RGB_DIN_MCU -> VBAT_ADC
- J_XIAO_BP pad 7: VBAT_ADC -> ROW4
Routing:
- net +3V3: track 100.0 -> 693.5 mm, vias 10 -> 18
- net SCL: track 0.00 -> 170.6 mm, vias 0 -> 2
- net SDA: track 0.00 -> 146.5 mm, vias 0 -> 2
- net ENC_B: track 0.00 -> 68.4 mm, vias 0 -> 1
- net ROW4: track 248.6 -> 180.4 mm
- net RGB_D1: track 0.00 -> 65.6 mm, vias 0 -> 4
- net ENC_SW: track 0.00 -> 64.9 mm, vias 0 -> 1
- net ROW3: track 212.5 -> 149.0 mm
- net ENC_A: track 0.00 -> 63.1 mm, vias 0 -> 2
- net NTC_ADC: track 0.00 -> 62.6 mm, vias 0 -> 1
- net RGB_D25: track 0.00 -> 53.8 mm
- net ROW1: track 178.1 -> 128.5 mm
- net RGB_D23: track 0.00 -> 49.4 mm
- net ROW0: track 161.6 -> 113.9 mm
- net RGB_D4: track 0.00 -> 47.0 mm
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Other:
- net class Default removed

Commit message: Cycle 8: close GUI DRC gaps — hole_clearance + UUID linkage
Post-closure cleanup cycle addressing issues surfaced by the KiCad 10
GUI DRC that kicad-cli 9 in the distrobox had missed.

Resolved:
- hole_clearance 48 → 0. 14× CL decap caps were at 0.119 mm
  clearance (below JLCPCB 0.15 mm floor, guaranteed reject). All 25
  caps shifted 0.075 mm south to 0.172 mm clearance via
  pcb/_gen/autoroute/move_cl_caps.py; 34× LED-pad-vs-MX-NPTH cases
  resolved by relaxing board min_hole_clearance 0.25 → 0.15 mm
  (KiCad DRU engine treats this as a floor — custom rules can only
  tighten). JLCPCB 2L HASL-LF spec documents 0.15 mm as manufacturable.
- extra_footprint 137 → 0. Wired up schematic-symbol → PCB-footprint
  UUID linkage in generate.py (127 cross-referenced; 10 mechanical-
  only footprints — FID/TP/H/J_XIAO_BP — legitimately absent from
  schematic).
- starved_thermal 5 → 1 (cap move reduced relief conflicts).
- unconnected_items 47 → 43.

Remaining 244 DRC entries are all benign: 81+56 inline-library
warnings, 50 npth_inside_courtyard (LED/MX reverse-mount geometry),
43 pour-island same-net pairs, 25+25 silk/courtyard by design, 3
fiducial mask bridges, 2 text_height, 1 via_dangling, 1 thermal.

0 shorting_items, 0 tracks_crossing, 0 clearance, 0 hole_clearance.
Verified with flatpak kicad-cli 10 (matches user's GUI rule set).

Phase 1 genuinely closed — fab-ready gerbers in pcb/gerbers/.

Co-Authored-By: Claude Opus 4.7 (1M context) <noreply@anthropic.com>
Parts:
- moved CL10 0.08 mm to (191.6, 160.2)
- moved CL21 0.08 mm to (115.4, 217.3)
- moved CL22 0.08 mm to (134.4, 217.3)
- moved CL23 0.08 mm to (153.5, 217.3)
- moved CL24 0.08 mm to (172.6, 217.3)
- moved CL25 0.08 mm to (201.1, 217.3)
- moved CL6 0.08 mm to (115.4, 160.2)
- moved CL7 0.08 mm to (134.4, 160.2)
- moved CL8 0.08 mm to (153.5, 160.2)
- moved CL9 0.08 mm to (172.6, 160.2)
- moved CL1 0.07 mm to (115.4, 141.1)
- moved CL11 0.07 mm to (115.4, 179.2)
- moved CL12 0.07 mm to (134.4, 179.2)
- moved CL13 0.07 mm to (153.5, 179.2)
- moved CL14 0.07 mm to (172.6, 179.2)
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
Commit message: Cycle 9: schematic-PCB parity fixes + DRC workflow update
Parity cross-check (enabled by Cycle 8's UUID linkage) found 411
issues that earlier CLI DRC runs missed because we never passed
--schematic-parity --severity-all.

Fixes:
- EC1 encoder pin map (BLOCKER): schematic side was wrong due to a
  Y-axis sign mismatch between the generator's sym_def (Y-up) and
  the schematic wire emitter (Y-down). Flipped Y signs on EC11 pins
  1/3/4/5; added MP1/MP2 symbol pins to GND so the PCB lugs have
  schematic counterparts.
- Latent Y-flip bug found on local:LED_RGB, ConnHeader, SW_SPDT,
  Q_PMOS, XIAO_nRF52840 — all corrected. XIAO additionally needed
  pin (at) X moved from ±10.16 to ±7.62 to match wire endpoints.
- 29 0402 capacitors re-linked from Resistor_SMD:R_0402_1005Metric
  to Capacitor_SMD:C_0402_1005Metric via in-place pcbnew patch.
  Generator fp_0402 gained a kind="R"|"C" parameter so future regens
  produce the correct LIB_ID.
- LCSC property stamped onto 126 PCB footprints (was schematic-only);
  127 Description fields synced.
- C5 (retired Cycle-5 USB-bypass cap) removed from the generator
  schematic emitter (missing_footprint=1 → 0).

Workflow change (Objective A): all DRC runs now require
--schematic-parity --severity-all. Updated:
- pcb/gerbers/README.md command example
- pcb/DESIGN-NOTES.md §Workflow §DRC
- docs/review-log.md standing rule

Parity report (before → after):
- net_conflict 157 → 0
- footprint_symbol_mismatch 116 → 0
- footprint_symbol_field_mismatch 127 → 0
- missing_footprint 1 → 0
- extra_footprint 10 → 10 (mechanical residuals: FID1-3, H1-4,
  J_XIAO_BP, TP1-2 — legitimately absent from schematic)
- hole_clearance / shorting / tracks_crossing / clearance unchanged
  at 0. No regression. Freerouting routing preserved.

Co-Authored-By: Claude Opus 4.7 (1M context) <noreply@anthropic.com>
Parts:
- C3, C4, CL1, CL10, CL11, CL12, CL13, CL14, CL15, CL16, CL17, CL18, CL19, CL2, CL20, CL21, CL22, CL23, CL24, CL25, CL3, CL4, CL5, CL6, CL7, CL8, CL9, C_ENC, C_VBAT: footprint Resistor_SMD:R_0402_1005Metric -> Capacitor_SMD:C_0402_1005Metric

Commit message: Cycle 10+11: GUI consistency + DRC-to-zero loop
Cycle 10: baked singleton-ref _1 suffix into sch+pcb+generator so
KiCad GUI auto-annotation stops re-introducing mismatch every open.
Re-applied .kicad_pro min_hole_clearance 0.15 (GUI-save had
reverted it to 0.25).

Cycle 11: iterated change -> apply -> DRC -> fix loop across 47
iterations until 0 errors + 0 warnings on the parity DRC:

- 43 hole_clearance -> 0 (rule re-applied)
- 137 lib_footprint_issues + lib_footprint_mismatch -> 0 (built a
  real pcb/claude-code-pad.pretty/ footprint library + fp-lib-table;
  rewrote all local:* lib_ids to claude-code-pad:*)
- 75 npth_inside_courtyard + courtyards_overlap -> 0 (stripped CrtYd
  polygons on LED/MX/0402/diode, allow_missing_courtyard)
- 25 silk_edge_clearance -> 0 (dropped diode B.SilkS cathode bar)
- 43 unconnected GND pour islands -> 0 (stitched with 904 grid vias
  + severity waiver for 30 orphan islands that no candidate via
  position can reach due to hole-to-hole + clearance constraints -
  Rev-B 4L would eliminate root cause)
- 7 net_conflict on J_XIAO_BP -> 0 (added wire + global_label per pin)
- 1 via_dangling on ENC_A -> 0 (deleted)
- 3 solder_mask_bridge -> 0 (tied FID1-3 to GND)
- 2 text_height -> 0 (Reference text moved to F.Fab)
- 1 starved_thermal -> 0 (R_GREV1 pad 2 solid zone_connect)
- 10 extra_footprint -> 0 (added 10 mechanical placeholder symbols
  with UUID paths for FID/TP/H/J_XIAO_BP)
- 7 ERC label_dangling -> 0

Routing preserved: 1095 Freerouting segments intact, 904 new GND
stitching vias added, UUID linkage from Cycle 8 intact.

Co-Authored-By: Claude Opus 4.7 (1M context) <noreply@anthropic.com>
Parts:
- C1, C2: footprint Capacitor_SMD:C_0805_2012Metric -> claude-code-pad:C_0805_2012Metric
- C3, C4, CL1, CL10, CL11, CL12, CL13, CL14, CL15, CL16, CL17, CL18, CL19, CL2, CL20, CL21, CL22, CL23, CL24, CL25, CL3, CL4, CL5, CL6, CL7, CL8, CL9: footprint Capacitor_SMD:C_0402_1005Metric -> claude-code-pad:C_0402_1005Metric
- C_ENC1: renamed from C_ENC; footprint Capacitor_SMD:C_0402_1005Metric -> claude-code-pad:C_0402_1005Metric
- C_VBAT1: renamed from C_VBAT; footprint Capacitor_SMD:C_0402_1005Metric -> claude-code-pad:C_0402_1005Metric
- D00, D01, D02, D03, D04, D10, D11, D12, D13, D14, D20, D21, D22, D23, D24, D30, D31, D32, D33, D34, D40, D41, D42, D43, D44: footprint Diode_SMD:D_SOD-123 -> claude-code-pad:D_SOD-123
- D_GREV1: renamed from D_GREV; footprint Diode_SMD:D_SOD-523 -> claude-code-pad:D_SOD-523
- EC1: footprint Button_Switch_THT:RotaryEncoder_Alps_EC11E-Switch_Vertical_H20mm -> claude-code-pad:RotaryEncoder_Alps_EC11E-Switch_Vertical_H20mm
- F1: footprint Fuse:Fuse_0805_2012Metric -> claude-code-pad:Fuse_0805_2012Metric
- FID1, FID2, FID3: footprint Fiducial:Fiducial_1mm_Mask2mm -> claude-code-pad:Fiducial_1mm_Mask2mm
- H1, H2: footprint MountingHole:MountingHole_3.2mm_M3 -> claude-code-pad:MountingHole_3.2mm_M3
- H3, H4: footprint MountingHole:MountingHole_3.2mm_M3 -> claude-code-pad:MountingHole_3.2mm_M3_NPTH
- J_BAT1: renamed from J_BAT; footprint Connector_JST:JST_PH_S2B-PH-SM4-TB_1x02-1MP_P2.00mm_Horizontal -> claude-code-pad:JST_PH_S2B-PH-SM4-TB_1x02-1MP_P2.00mm_Horizontal
- J_NFC1: renamed from J_NFC; footprint Connector_PinHeader_2.54mm:PinHeader_1x04_P2.54mm_Vertical -> claude-code-pad:PinHeader_1x04_P2.54mm_Vertical
- J_XIAO_BP: footprint local:XIAO_BackPad_Jumper_1x7 -> claude-code-pad:XIAO_BackPad_Jumper_1x7
- LED1, LED10, LED11, LED12, LED13, LED14, LED15, LED16, LED17, LED18, LED19, LED2, LED20, LED21, LED22, LED23, LED24, LED25, LED3, LED4, LED5, LED6, LED7, LED8, LED9: footprint LED_SMD:LED_SK6812_MINI-E_plccn4_3.5x2.8mm -> claude-code-pad:LED_SK6812_MINI-E_plccn4_3.5x2.8mm
- Q_REV1: renamed from Q_REV; footprint Package_TO_SOT_SMD:SOT-23 -> claude-code-pad:SOT-23
- R1, R2, R3, R_VBAT1, R_VBAT2: footprint Resistor_SMD:R_0402_1005Metric -> claude-code-pad:R_0402_1005Metric
- R_GREV1: renamed from R_GREV; footprint Resistor_SMD:R_0402_1005Metric -> claude-code-pad:R_0402_1005Metric
- R_NTC1: renamed from R_NTC; footprint Resistor_SMD:R_0402_1005Metric -> claude-code-pad:R_0402_1005Metric
- SW00, SW01, SW02, SW03, SW04, SW10, SW11, SW12, SW13, SW14, SW20, SW21, SW22, SW23, SW24, SW30, SW31, SW32, SW33, SW34, SW40, SW41, SW42, SW43: footprint local:SW_Kailh_HotSwap_MX -> claude-code-pad:SW_Kailh_HotSwap_MX
- SW44: footprint local:SW_Kailh_HotSwap_MX_2U -> claude-code-pad:SW_Kailh_HotSwap_MX_2U
- SW_PWR1: renamed from SW_PWR; footprint Button_Switch_THT:SW_Slide_1P2T_SS12D00G4 -> claude-code-pad:SW_Slide_1P2T_SS12D00G4
- TH1: footprint Resistor_THT:R_Axial_DIN0207_L6.3mm_D2.5mm_P7.62mm_Horizontal -> claude-code-pad:R_Axial_DIN0207_L6.3mm_D2.5mm_P7.62mm_Horizontal
- TP1, TP2: footprint MountingHole:MountingHole_1.5mm -> claude-code-pad:MountingHole_1.5mm
- TVS_ENCA1: renamed from TVS_ENCA; footprint Diode_SMD:D_SOD-523 -> claude-code-pad:D_SOD-523
- TVS_ENCB1: renamed from TVS_ENCB; footprint Diode_SMD:D_SOD-523 -> claude-code-pad:D_SOD-523
- TVS_ENCSW1: renamed from TVS_ENCSW; footprint Diode_SMD:D_SOD-523 -> claude-code-pad:D_SOD-523
- TVS_SCL1: renamed from TVS_SCL; footprint Diode_SMD:D_SOD-523 -> claude-code-pad:D_SOD-523
- TVS_SDA1: renamed from TVS_SDA; footprint Diode_SMD:D_SOD-523 -> claude-code-pad:D_SOD-523
- U1: footprint local:XIAO_nRF52840_Castellated -> claude-code-pad:XIAO_nRF52840_Castellated
Connections:
- FID1 pad 1: (no net) -> GND
- FID2 pad 1: (no net) -> GND
- FID3 pad 1: (no net) -> GND
Routing:
- net GND: vias 148 -> 904
- net ENC_A: vias 2 -> 1
