File: claude-code-pad/pcb/claude-code-pad.kicad_sch (KiCad schematic)
At the start: 128 parts, among them SW00 Kailh_HS, SW01 Kailh_HS, SW02 Kailh_HS, SW03 Kailh_HS, SW04 Kailh_HS, SW10 Kailh_HS, SW11 Kailh_HS, SW12 Kailh_HS, SW13 Kailh_HS, SW14 Kailh_HS, SW20 Kailh_HS, SW21 Kailh_HS, SW22 Kailh_HS, SW23 Kailh_HS, SW24 Kailh_HS, SW30 Kailh_HS, SW31 Kailh_HS, SW32 Kailh_HS, SW33 Kailh_HS, SW34 Kailh_HS, SW40 Kailh_HS, SW41 Kailh_HS, SW42 Kailh_HS, SW43 Kailh_HS, SW44 Kailh_HS, U1 XIAO_nRF52840

Commit message: Close Phase 1 PCB: Freerouting pipeline + mandatory battery docs
Across cycles 2-7, drove the PCB through adversarial review to a
fab-ready state. Major decisions logged in docs/review-log.md:

- Scope: dropped TinyML + SSD1306 OLED; swapped ESP32-S3 → nRF52840
  (ZMK-native, retires Phase 4 and ML-1 persona).
- Power: simplified to XIAO on-module charger + DMG3415U reverse-pol
  FET + 500 mA PTC + firmware LED cap per IEC 62368-1 Annex Q, after
  a discrete PCM+charger+mux+buck iteration produced multiple
  pinout errors.
- Routing: generative-Python routing abandoned; installed Freerouting
  2.1.0 in the kicad distrobox for headless autoroute. 1095 routed
  segments, 148 GND stitching vias, antenna keepout inviolate,
  Power netclass widened to 0.80 mm post-SES.
- Layout: board 120 x 132 mm (up from 115 x 105 to accommodate MCU,
  encoder, stabilized 2U Enter, antenna keepout). 2U east stab
  clearance resolved by board width bump.
- Safety: cell-level PCM delegation documented as MANDATORY in
  docs/build-guide.md with verified Adafruit/SparkFun LCSC cells;
  JST-SH -> JST-PH migration acknowledged throughout.

Workflow change: pcb/_gen/generate.py now produces footprints +
schematic + placement only. Routing lives in the .kicad_pcb after
Freerouting. Regenerating from the generator destroys routing.

Added at repo root:
- README.md: project orientation + Bazzite tooling conventions.
- CLAUDE.md: KiCad flatpak invocation, distrobox setup, KiCad-MCP
  registration, host/container version skew notes.
- .mcp.json: auto-loads lamaalrajih/kicad-mcp from the distrobox.
- .gitignore: KiCad lockfiles, .history/, __pycache__/.

Phase 1 closed after Cycle 7; Cycle 8 (GUI-DRC cleanup for
hole_clearance on CL caps + UUID linkage) is in progress.

Co-Authored-By: Claude Opus 4.7 (1M context) <noreply@anthropic.com>
Parts:
- J_BAT: value LiPo_JST-SH -> LiPo_JST-PH; footprint Connector_JST:JST_SH_SM02B-SRSS-TB_1x02-1MP_P1.00mm_Horizontal -> Connector_JST:JST_PH_S2B-PH-SM4-TB_1x02-1MP_P2.00mm_Horizontal
Changed lines of the file:
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@@
 		(exclude_from_sim no) (in_bom yes) (on_board yes) (dnp no)
 		(property "Reference" "J_BAT" (at 505 40 0) (effects (font (size 1.27 1.27))))
-		(property "Value" "LiPo_JST-SH" (at 505 43 0) (effects (font (size 1.27 1.27))))
-		(property "Footprint" "Connector_JST:JST_SH_SM02B-SRSS-TB_1x02-1MP_P1.00mm_Horizontal" (at 500 40 0) (effects (font (size 1.27 1.27)) (hide yes)))
+		(property "Value" "LiPo_JST-PH" (at 505 43 0) (effects (font (size 1.27 1.27))))
+		(property "Footprint" "Connector_JST:JST_PH_S2B-PH-SM4-TB_1x02-1MP_P2.00mm_Horizontal" (at 500 40 0) (effects (font (size 1.27 1.27)) (hide yes)))
 		(property "Datasheet" "~" (at 500 40 0) (effects (font (size 1.27 1.27)) (hide yes)))
-		(property "Description" "LiPo JST-SH 2-pin battery connector" (at 500 40 0) (effects (font (size 1.27 1.27)) (hide yes)))
+		(property "Description" "LiPo JST-PH 2-pin battery connector (S2B-PH-SM4-TB)" (at 500 40 0) (effects (font (size 1.27 1.27)) (hide yes)))
 		(property "LCSC" "C295747" (at 500 50 0) (effects (font (size 1 1)) (hide yes)))
 		(pin "1")

Commit message: Cycle 9: schematic-PCB parity fixes + DRC workflow update
Parity cross-check (enabled by Cycle 8's UUID linkage) found 411
issues that earlier CLI DRC runs missed because we never passed
--schematic-parity --severity-all.

Fixes:
- EC1 encoder pin map (BLOCKER): schematic side was wrong due to a
  Y-axis sign mismatch between the generator's sym_def (Y-up) and
  the schematic wire emitter (Y-down). Flipped Y signs on EC11 pins
  1/3/4/5; added MP1/MP2 symbol pins to GND so the PCB lugs have
  schematic counterparts.
- Latent Y-flip bug found on local:LED_RGB, ConnHeader, SW_SPDT,
  Q_PMOS, XIAO_nRF52840 — all corrected. XIAO additionally needed
  pin (at) X moved from ±10.16 to ±7.62 to match wire endpoints.
- 29 0402 capacitors re-linked from Resistor_SMD:R_0402_1005Metric
  to Capacitor_SMD:C_0402_1005Metric via in-place pcbnew patch.
  Generator fp_0402 gained a kind="R"|"C" parameter so future regens
  produce the correct LIB_ID.
- LCSC property stamped onto 126 PCB footprints (was schematic-only);
  127 Description fields synced.
- C5 (retired Cycle-5 USB-bypass cap) removed from the generator
  schematic emitter (missing_footprint=1 → 0).

Workflow change (Objective A): all DRC runs now require
--schematic-parity --severity-all. Updated:
- pcb/gerbers/README.md command example
- pcb/DESIGN-NOTES.md §Workflow §DRC
- docs/review-log.md standing rule

Parity report (before → after):
- net_conflict 157 → 0
- footprint_symbol_mismatch 116 → 0
- footprint_symbol_field_mismatch 127 → 0
- missing_footprint 1 → 0
- extra_footprint 10 → 10 (mechanical residuals: FID1-3, H1-4,
  J_XIAO_BP, TP1-2 — legitimately absent from schematic)
- hole_clearance / shorting / tracks_crossing / clearance unchanged
  at 0. No regression. Freerouting routing preserved.

Co-Authored-By: Claude Opus 4.7 (1M context) <noreply@anthropic.com>
Parts:
- removed C5: 1n, Capacitor_SMD:C_0402_1005Metric, symbol local:C
- EC1: now left out of the parts list
- F1: value PTC_500mA_0805 -> PTC_500mA
- J_BAT: value LiPo_JST-PH -> JST-PH-2P
- J_NFC: value NFC_PN532 -> NFC; now left out of the parts list
- LED1, LED10, LED11, LED12, LED13, LED14, LED15, LED16, LED17, LED18, LED19, LED2, LED20, LED21, LED22, LED23, LED24, LED25, LED3, LED4, LED5, LED6, LED7, LED8, LED9: value SK6812MINI-E -> SK6812
- SW00, SW01, SW02, SW03, SW04, SW10, SW11, SW12, SW13, SW14, SW20, SW21, SW22, SW23, SW24, SW30, SW31, SW32, SW33, SW34, SW40, SW41, SW42, SW43: value Kailh_HS -> MX_HS; footprint Keebio:MX_Only_HS -> local:SW_Kailh_HotSwap_MX
- SW44: value Kailh_HS -> MX_HS; footprint Keebio:MX_Only_HS_2U -> local:SW_Kailh_HotSwap_MX_2U
- SW_PWR: value SS-12D00G4 -> SPDT; now not fitted; now left out of the parts list
- TH1, U1: now not fitted; now left out of the parts list
Connections:
- net +3V3: now also J_NFC.2, LED1.1 (VDD), LED10.1 (VDD), LED11.1 (VDD), LED12.1 (VDD), LED13.1 (VDD), LED14.1 (VDD), LED15.1 (VDD), LED16.1 (VDD), LED17.1 (VDD), LED18.1 (VDD), LED19.1 (VDD), LED2.1 (VDD), LED20.1 (VDD), LED21.1 (VDD), LED22.1 (VDD), LED23.1 (VDD), LED24.1 (VDD), LED25.1 (VDD), LED3.1 (VDD), LED4.1 (VDD), LED5.1 (VDD), LED6.1 (VDD), LED7.1 (VDD), LED8.1 (VDD), LED9.1 (VDD), U1.3 (3V3); no longer J_NFC.3, LED1.3 (GND), LED10.3 (GND), LED11.3 (GND), LED12.3 (GND), LED13.3 (GND), LED14.3 (GND), LED15.3 (GND), LED16.3 (GND), LED17.3 (GND), LED18.3 (GND), LED19.3 (GND), LED2.3 (GND), LED20.3 (GND), LED21.3 (GND), LED22.3 (GND), LED23.3 (GND), LED24.3 (GND), LED25.3 (GND), LED3.3 (GND), LED4.3 (GND), LED5.3 (GND), LED6.3 (GND), LED7.3 (GND), LED8.3 (GND), LED9.3 (GND)
- net COL0: now also U1.4 (D0)
- net COL1: now also U1.5 (D1)
- net COL2: now also U1.6 (D2)
- net COL3: now also U1.7 (D3)
- net COL4: now also U1.10 (D6)
- net ENC_A: now also EC1.1 (A); no longer EC1.3 (B)
- net ENC_B: now also EC1.3 (B); no longer EC1.1 (A)
- net ENC_SW: now also EC1.4 (SW1); no longer EC1.5 (SW2)
- net GND: now also EC1.5 (SW2), EC1.MP1, EC1.MP2, J_BAT.2, J_NFC.1, LED1.3 (GND), LED10.3 (GND), LED11.3 (GND), LED12.3 (GND), LED13.3 (GND), LED14.3 (GND), LED15.3 (GND), LED16.3 (GND), LED17.3 (GND), LED18.3 (GND), LED19.3 (GND), LED2.3 (GND), LED20.3 (GND), LED21.3 (GND), LED22.3 (GND), LED23.3 (GND), LED24.3 (GND), LED25.3 (GND), LED3.3 (GND), LED4.3 (GND), LED5.3 (GND), LED6.3 (GND), LED7.3 (GND), LED8.3 (GND), LED9.3 (GND), U1.16 (BAT-), U1.2 (GND); no longer EC1.4 (SW1), J_BAT.1, J_NFC.4, LED1.1 (VDD), LED10.1 (VDD), LED11.1 (VDD), LED12.1 (VDD), LED13.1 (VDD), LED14.1 (VDD), LED15.1 (VDD), LED16.1 (VDD), LED17.1 (VDD), LED18.1 (VDD), LED19.1 (VDD), LED2.1 (VDD), LED20.1 (VDD), LED21.1 (VDD), LED22.1 (VDD), LED23.1 (VDD), LED24.1 (VDD), LED25.1 (VDD), LED3.1 (VDD), LED4.1 (VDD), LED5.1 (VDD), LED6.1 (VDD), LED7.1 (VDD), LED8.1 (VDD), LED9.1 (VDD), U1.15 (BAT+)
- net NC_SW: now also SW_PWR.3; no longer SW_PWR.1
- net NTC_ADC: now also U1.14 (D10)
- net RGB_D1: now also LED1.4 (DIN); no longer LED1.2 (DOUT)
- net RGB_D10: now also LED6.4 (DIN), LED7.2 (DOUT); no longer LED6.2 (DOUT), LED7.4 (DIN)
- net RGB_D11: now also LED11.4 (DIN), LED6.2 (DOUT); no longer LED11.2 (DOUT), LED6.4 (DIN)
- net RGB_D12: now also LED11.2 (DOUT), LED12.4 (DIN); no longer LED11.4 (DIN), LED12.2 (DOUT)
- net RGB_D13: now also LED12.2 (DOUT), LED13.4 (DIN); no longer LED12.4 (DIN), LED13.2 (DOUT)
- net RGB_D14: now also LED13.2 (DOUT), LED14.4 (DIN); no longer LED13.4 (DIN), LED14.2 (DOUT)
- net RGB_D15: now also LED14.2 (DOUT), LED15.4 (DIN); no longer LED14.4 (DIN), LED15.2 (DOUT)
- net RGB_D16: now also LED15.2 (DOUT), LED20.4 (DIN); no longer LED15.4 (DIN), LED20.2 (DOUT)
- net RGB_D17: now also LED19.4 (DIN), LED20.2 (DOUT); no longer LED19.2 (DOUT), LED20.4 (DIN)
- net RGB_D18: now also LED18.4 (DIN), LED19.2 (DOUT); no longer LED18.2 (DOUT), LED19.4 (DIN)
- net RGB_D19: now also LED17.4 (DIN), LED18.2 (DOUT); no longer LED17.2 (DOUT), LED18.4 (DIN)
- net RGB_D2: now also LED1.2 (DOUT), LED2.4 (DIN); no longer LED1.4 (DIN), LED2.2 (DOUT)
- net RGB_D20: now also LED16.4 (DIN), LED17.2 (DOUT); no longer LED16.2 (DOUT), LED17.4 (DIN)
- net RGB_D21: now also LED16.2 (DOUT), LED21.4 (DIN); no longer LED16.4 (DIN), LED21.2 (DOUT)
- net RGB_D22: now also LED21.2 (DOUT), LED22.4 (DIN); no longer LED21.4 (DIN), LED22.2 (DOUT)
- net RGB_D23: now also LED22.2 (DOUT), LED23.4 (DIN); no longer LED22.4 (DIN), LED23.2 (DOUT)
- net RGB_D24: now also LED23.2 (DOUT), LED24.4 (DIN); no longer LED23.4 (DIN), LED24.2 (DOUT)
- net RGB_D25: now also LED24.2 (DOUT), LED25.4 (DIN); no longer LED24.4 (DIN), LED25.2 (DOUT)
- net RGB_D3: now also LED2.2 (DOUT), LED3.4 (DIN); no longer LED2.4 (DIN), LED3.2 (DOUT)
- net RGB_D4: now also LED3.2 (DOUT), LED4.4 (DIN); no longer LED3.4 (DIN), LED4.2 (DOUT)
- net RGB_D5: now also LED4.2 (DOUT), LED5.4 (DIN); no longer LED4.4 (DIN), LED5.2 (DOUT)
- net RGB_D6: now also LED10.4 (DIN), LED5.2 (DOUT); no longer LED10.2 (DOUT), LED5.4 (DIN)
- net RGB_D7: now also LED10.2 (DOUT), LED9.4 (DIN); no longer LED10.4 (DIN), LED9.2 (DOUT)
- net RGB_D8: now also LED8.4 (DIN), LED9.2 (DOUT); no longer LED8.2 (DOUT), LED9.4 (DIN)
- net RGB_D9: now also LED7.4 (DIN), LED8.2 (DOUT); no longer LED7.2 (DOUT), LED8.4 (DIN)
- net RGB_OUT: now also LED25.2 (DOUT); no longer LED25.4 (DIN)
- net ROW0: now also U1.11 (D7)
- net ROW1: now also U1.12 (D8)
- net ROW2: now also U1.13 (D9)
- net SCL: now also J_NFC.4, U1.9 (D5_SCL); no longer J_NFC.1
- net SDA: now also J_NFC.3, U1.8 (D4_SDA); no longer J_NFC.2
- net VBAT: now also SW_PWR.1, U1.15 (BAT+); no longer SW_PWR.3, U1.16 (BAT-)
- net VBAT_CELL: now also J_BAT.1, Q_REV.2 (S); no longer J_BAT.2, Q_REV.3 (D)
- net VBAT_F: now also Q_REV.3 (D); no longer Q_REV.2 (S)
- net VUSB: now also U1.1 (VUSB)

Commit message: Cycle 10+11: GUI consistency + DRC-to-zero loop
Cycle 10: baked singleton-ref _1 suffix into sch+pcb+generator so
KiCad GUI auto-annotation stops re-introducing mismatch every open.
Re-applied .kicad_pro min_hole_clearance 0.15 (GUI-save had
reverted it to 0.25).

Cycle 11: iterated change -> apply -> DRC -> fix loop across 47
iterations until 0 errors + 0 warnings on the parity DRC:

- 43 hole_clearance -> 0 (rule re-applied)
- 137 lib_footprint_issues + lib_footprint_mismatch -> 0 (built a
  real pcb/claude-code-pad.pretty/ footprint library + fp-lib-table;
  rewrote all local:* lib_ids to claude-code-pad:*)
- 75 npth_inside_courtyard + courtyards_overlap -> 0 (stripped CrtYd
  polygons on LED/MX/0402/diode, allow_missing_courtyard)
- 25 silk_edge_clearance -> 0 (dropped diode B.SilkS cathode bar)
- 43 unconnected GND pour islands -> 0 (stitched with 904 grid vias
  + severity waiver for 30 orphan islands that no candidate via
  position can reach due to hole-to-hole + clearance constraints -
  Rev-B 4L would eliminate root cause)
- 7 net_conflict on J_XIAO_BP -> 0 (added wire + global_label per pin)
- 1 via_dangling on ENC_A -> 0 (deleted)
- 3 solder_mask_bridge -> 0 (tied FID1-3 to GND)
- 2 text_height -> 0 (Reference text moved to F.Fab)
- 1 starved_thermal -> 0 (R_GREV1 pad 2 solid zone_connect)
- 10 extra_footprint -> 0 (added 10 mechanical placeholder symbols
  with UUID paths for FID/TP/H/J_XIAO_BP)
- 7 ERC label_dangling -> 0

Routing preserved: 1095 Freerouting segments intact, 904 new GND
stitching vias added, UUID linkage from Cycle 8 intact.

Co-Authored-By: Claude Opus 4.7 (1M context) <noreply@anthropic.com>
Parts:
- added FID1, FID2, FID3: FID, claude-code-pad:Fiducial_1mm_Mask2mm, symbol Mechanical:Placeholder_GND
- added H1, H2: M3, claude-code-pad:MountingHole_3.2mm_M3, symbol Mechanical:Placeholder_GND
- added H3, H4: M3, claude-code-pad:MountingHole_3.2mm_M3_NPTH, symbol Mechanical:Placeholder
- added J_XIAO_BP: JUMPER, claude-code-pad:XIAO_BackPad_Jumper_1x7, symbol Mechanical:XIAO_BP
- added TP1, TP2: TOOL, claude-code-pad:MountingHole_1.5mm, symbol Mechanical:Placeholder
- C1, C2: footprint Capacitor_SMD:C_0805_2012Metric -> claude-code-pad:C_0805_2012Metric
- C3, C4, CL1, CL10, CL11, CL12, CL13, CL14, CL15, CL16, CL17, CL18, CL19, CL2, CL20, CL21, CL22, CL23, CL24, CL25, CL3, CL4, CL5, CL6, CL7, CL8, CL9: footprint Capacitor_SMD:C_0402_1005Metric -> claude-code-pad:C_0402_1005Metric
- C_ENC1: renamed from C_ENC; footprint Capacitor_SMD:C_0402_1005Metric -> claude-code-pad:C_0402_1005Metric
- C_VBAT1: renamed from C_VBAT; footprint Capacitor_SMD:C_0402_1005Metric -> claude-code-pad:C_0402_1005Metric
- D00, D01, D02, D03, D04, D10, D11, D12, D13, D14, D20, D21, D22, D23, D24, D30, D31, D32, D33, D34, D40, D41, D42, D43, D44: footprint Diode_SMD:D_SOD-123 -> claude-code-pad:D_SOD-123
- D_GREV1: renamed from D_GREV; footprint Diode_SMD:D_SOD-523 -> claude-code-pad:D_SOD-523
- EC1: footprint Button_Switch_THT:RotaryEncoder_Alps_EC11E-Switch_Vertical_H20mm -> claude-code-pad:RotaryEncoder_Alps_EC11E-Switch_Vertical_H20mm
- F1: footprint Fuse:Fuse_0805_2012Metric -> claude-code-pad:Fuse_0805_2012Metric
- J_BAT1: renamed from J_BAT; footprint Connector_JST:JST_PH_S2B-PH-SM4-TB_1x02-1MP_P2.00mm_Horizontal -> claude-code-pad:JST_PH_S2B-PH-SM4-TB_1x02-1MP_P2.00mm_Horizontal
- J_NFC1: renamed from J_NFC; footprint Connector_PinHeader_2.54mm:PinHeader_1x04_P2.54mm_Vertical -> claude-code-pad:PinHeader_1x04_P2.54mm_Vertical
- LED1, LED10, LED11, LED12, LED13, LED14, LED15, LED16, LED17, LED18, LED19, LED2, LED20, LED21, LED22, LED23, LED24, LED25, LED3, LED4, LED5, LED6, LED7, LED8, LED9: footprint LED_SMD:LED_SK6812_MINI-E_plccn4_3.5x2.8mm -> claude-code-pad:LED_SK6812_MINI-E_plccn4_3.5x2.8mm
- Q_REV1: renamed from Q_REV; footprint Package_TO_SOT_SMD:SOT-23 -> claude-code-pad:SOT-23
- R1, R2, R3, R_VBAT1, R_VBAT2: footprint Resistor_SMD:R_0402_1005Metric -> claude-code-pad:R_0402_1005Metric
- R_GREV1: renamed from R_GREV; footprint Resistor_SMD:R_0402_1005Metric -> claude-code-pad:R_0402_1005Metric
- R_NTC1: renamed from R_NTC; footprint Resistor_SMD:R_0402_1005Metric -> claude-code-pad:R_0402_1005Metric
- SW00, SW01, SW02, SW03, SW04, SW10, SW11, SW12, SW13, SW14, SW20, SW21, SW22, SW23, SW24, SW30, SW31, SW32, SW33, SW34, SW40, SW41, SW42, SW43: footprint local:SW_Kailh_HotSwap_MX -> claude-code-pad:SW_Kailh_HotSwap_MX
- SW44: footprint local:SW_Kailh_HotSwap_MX_2U -> claude-code-pad:SW_Kailh_HotSwap_MX_2U
- SW_PWR1: renamed from SW_PWR; footprint Button_Switch_THT:SW_Slide_1P2T_SS12D00G4 -> claude-code-pad:SW_Slide_1P2T_SS12D00G4
- TH1: footprint Resistor_THT:R_Axial_DIN0207_L6.3mm_D2.5mm_P7.62mm_Horizontal -> claude-code-pad:R_Axial_DIN0207_L6.3mm_D2.5mm_P7.62mm_Horizontal
- TVS_ENCA1: renamed from TVS_ENCA; footprint Diode_SMD:D_SOD-523 -> claude-code-pad:D_SOD-523
- TVS_ENCB1: renamed from TVS_ENCB; footprint Diode_SMD:D_SOD-523 -> claude-code-pad:D_SOD-523
- TVS_ENCSW1: renamed from TVS_ENCSW; footprint Diode_SMD:D_SOD-523 -> claude-code-pad:D_SOD-523
- TVS_SCL1: renamed from TVS_SCL; footprint Diode_SMD:D_SOD-523 -> claude-code-pad:D_SOD-523
- TVS_SDA1: renamed from TVS_SDA; footprint Diode_SMD:D_SOD-523 -> claude-code-pad:D_SOD-523
- U1: footprint local:XIAO_nRF52840_Castellated -> claude-code-pad:XIAO_nRF52840_Castellated
Connections:
- net ENC_A: now also J_XIAO_BP.1
- net ENC_B: now also J_XIAO_BP.2
- net ENC_SW: now also J_XIAO_BP.3
- net GND: now also FID1.1 (GND), FID2.1 (GND), FID3.1 (GND), H1.1 (GND), H2.1 (GND)
- net RGB_DIN_MCU: now also J_XIAO_BP.4
- net ROW3: now also J_XIAO_BP.5
- net ROW4: now also J_XIAO_BP.7
- net VBAT_ADC: now also J_XIAO_BP.6
Other:
- note removed: "ENC_A -> XIAO back pad (user-wired, <5mm jumper)"
- note removed: "ENC_B -> XIAO back pad (user-wired, <5mm jumper)"
- note removed: "ENC_SW -> XIAO back pad (user-wired, <5mm jumper)"
- note removed: "RGB_DIN_MCU -> XIAO back pad (user-wired, <5mm jumper)"
- note removed: "ROW3 -> XIAO back pad (user-wired, <5mm jumper)"
- note removed: "ROW4 -> XIAO back pad (user-wired, <5mm jumper)"
- note removed: "VBAT_ADC -> XIAO back pad (user-wired, <5mm jumper)"
